Commit message: New moveit config for 7dof; nimbus_bringup not yet updated, but motion planning will work if you launch the required nodes individually

File: nimbus_description/urdf/structure/arm_mount.urdf.xacro (robot description, xacro)
@@ -31,5 +31,5 @@
       <parent link="arm_mount_plate_link" />
       <child link="arm_mount_beam_link" />
-      <origin xyz="0 0 0" rpy="0 0 ${pi}" />
+      <origin xyz="0 0 0" rpy="0 0 0" />
     </joint>
     <link name="arm_mount_beam_link">
@@ -48,5 +48,11 @@
       </collision>
     </link>
-    <xacro:j2s7s300 base_parent="arm_mount_beam_link"></xacro:j2s7s300>
+    <joint name="arm_mount_beam_link_arm_mount_offset_link_joint" type="fixed">
+      <parent link="arm_mount_beam_link" />
+      <child link="arm_mount_offset_link" />
+      <origin xyz="0 0 0.0508" rpy="0 0 ${pi}" />
+    </joint>
+    <link name="arm_mount_offset_link" />
+    <xacro:j2s7s300 base_parent="arm_mount_offset_link" />
     <joint name="jaco_ee_link_nimbus_ee_link_joint" type="fixed">
       <parent link="j2s7s300_ee_link" />

Commit message: Nimbus ee link fix and re-generated moveit config files

File: nimbus_description/urdf/structure/arm_mount.urdf.xacro (robot description, xacro)
@@ -58,5 +58,5 @@
       <parent link="j2s7s300_ee_link" />
       <child link="nimbus_ee_link" />
-      <origin xyz="0 0 0" rpy="0 ${-pi/2.0} 0" />
+      <origin xyz="0 0 0" rpy="${pi/2.0} 0 0" />
     </joint>
     <link name="nimbus_ee_link" />
