Commit message: Updated launch files, vision packages, and robot model for use with the xtion instead of the kinect v2

File: nimbus_description/robots/nimbus.urdf (robot description, URDF)
Before this commit: robot nimbus, 48 links, 47 joints
Links:
- removed link kinect2_link
- removed link kinect2_mic_bar_link
- removed link kinect2_mounting_plate_link
- removed link kinect2_structure_link
- removed link kinect2_tilt_base_link
- removed link kinect2_tilt_link
- removed link sensor_frame_camera_plate_link
- removed link sensor_frame_camera_strut_link
- added link camera_depth_frame
- added link camera_depth_optical_frame
- added link camera_link, mass 0.170; collision box size=0.0730 0.2760 0.0720; visual mesh filename=package://nimbus_description/meshes/xtion_pro_camera.dae
- added link camera_rgb_frame
- added link camera_rgb_optical_frame
Joints:
- removed joint kinect2_mic_bar_link_kinect2_tilt_base_link_joint
- removed joint kinect2_mounting_plate_link_kinect2_mic_bar_link_joint
- removed joint kinect2_structure_link_kinect2_link_joint
- removed joint kinect2_tilt_base_link_kinect2_tilt_link_joint
- removed joint kinect2_tilt_link_kinect2_structure_link_joint
- removed joint sensor_frame_camera_plate_link_sensor_frame_sensor_link_joint
- removed joint sensor_frame_camera_strut_link_sensor_frame_camera_plate_link_joint
- removed joint sensor_frame_sensor_link_kinect2_mounting_plate_link_joint
- removed joint sensor_frame_top_beam_link_sensor_frame_camera_strut_link_joint
- added joint camera_depth_joint: type fixed, parent camera_rgb_frame, child camera_depth_frame, origin xyz=0 0.027 0 rpy=0 0 0
- added joint camera_depth_optical_joint: type fixed, parent camera_depth_frame, child camera_depth_optical_frame, origin xyz=0 0 0 rpy=-1.57079632679 0 -1.57079632679
- added joint camera_joint: type fixed, parent camera_rgb_frame, child camera_link, origin xyz=0 -0.022 0 rpy=0 0 0
- added joint camera_rgb_joint: type fixed, parent sensor_frame_sensor_link, child camera_rgb_frame, origin xyz=0.023 -0.014 -0.04 rpy=0.0 -0.223 0.0
- added joint camera_rgb_optical_joint: type fixed, parent camera_rgb_frame, child camera_rgb_optical_frame, origin xyz=0 0 0 rpy=-1.57079632679 0 -1.57079632679
- added joint sensor_frame_top_beam_link_sensor_frame_sensor_link_joint: type fixed, parent sensor_frame_top_beam_link, child sensor_frame_sensor_link, origin xyz=0.0 0.07 -0.038 rpy=0 1.57079632679 1.57079632679

File: nimbus_description/robots/nimbus_calibration.urdf (robot description, URDF)
Before this commit: robot nimbus, 53 links, 52 joints
Links:
- removed link kinect2_link
- removed link kinect2_mic_bar_link
- removed link kinect2_mounting_plate_link
- removed link kinect2_structure_link
- removed link kinect2_tilt_base_link
- removed link kinect2_tilt_link
- removed link sensor_frame_camera_plate_link
- removed link sensor_frame_camera_strut_link
- added link camera_depth_frame
- added link camera_depth_optical_frame
- added link camera_link, mass 0.170; collision box size=0.0730 0.2760 0.0720; visual mesh filename=package://nimbus_description/meshes/xtion_pro_camera.dae
- added link camera_rgb_frame
- added link camera_rgb_optical_frame
- added link sensor_frame_sensor_pitch_link
Joints:
- removed joint kinect2_mic_bar_link_kinect2_tilt_base_link_joint
- removed joint kinect2_mounting_plate_link_kinect2_mic_bar_link_joint
- removed joint kinect2_structure_link_kinect2_link_joint
- removed joint kinect2_tilt_base_link_kinect2_tilt_link_joint
- removed joint kinect2_tilt_link_kinect2_structure_link_joint
- removed joint sensor_frame_camera_plate_link_sensor_frame_sensor_calibration_link_joint
- removed joint sensor_frame_camera_strut_link_sensor_frame_camera_plate_link_joint
- removed joint sensor_frame_sensor_link_kinect2_mounting_plate_link_joint
- removed joint sensor_frame_top_beam_link_sensor_frame_camera_strut_link_joint
- added joint camera_depth_joint: type fixed, parent camera_rgb_frame, child camera_depth_frame, origin xyz=0 0.027 0 rpy=0 0 0
- added joint camera_depth_optical_joint: type fixed, parent camera_depth_frame, child camera_depth_optical_frame, origin xyz=0 0 0 rpy=-1.57079632679 0 -1.57079632679
- added joint camera_joint: type fixed, parent camera_rgb_frame, child camera_link, origin xyz=0 -0.022 0 rpy=0 0 0
- added joint camera_rgb_joint: type fixed, parent sensor_frame_sensor_link, child camera_rgb_frame, origin xyz=0.0 0.0 0.0 rpy=0.0 0.0 0.0
- added joint camera_rgb_optical_joint: type fixed, parent camera_rgb_frame, child camera_rgb_optical_frame, origin xyz=0 0 0 rpy=-1.57079632679 0 -1.57079632679
- added joint sensor_frame_sensor_calibrate_pitch: type revolute, parent sensor_frame_sensor_z_link, child sensor_frame_sensor_pitch_link, axis 0 1 0, limit lower=0.392699081699 upper=-0.392699081699 effort=100 velocity=20
- added joint sensor_frame_top_beam_link_sensor_frame_sensor_calibration_link_joint: type fixed, parent sensor_frame_top_beam_link, child sensor_frame_sensor_calibration_link, origin xyz=0.0 0.07 -0.038 rpy=0 1.57079632679 1.57079632679
- joint sensor_frame_sensor_calibrate_yaw: parent sensor_frame_sensor_z_link -> sensor_frame_sensor_pitch_link

File: nimbus_description/urdf/structure/sensor_structure.urdf.xacro (robot description, xacro)
@@ -4,5 +4,5 @@
        xmlns:interface="http://playerstage.sourceforge.net/gazebo/xmlschema/#interface"
        xmlns:xacro="http://ros.org/wiki/xacro">
-  <xacro:include filename="$(find nimbus_description)/urdf/sensors/kinect2.urdf.xacro" />
+  <xacro:include filename="$(find nimbus_description)/urdf/sensors/asus_xtion_pro.urdf.xacro" />
   <!-- Xacro properties -->
   <xacro:property name="pi" value="3.1415926535897931" />
@@ -11,13 +11,13 @@
       <xacro:insert_block name="origin" />
     </xacro:nimbus_sensor_frame_structure>
-    <joint name="sensor_frame_camera_plate_link_sensor_frame_sensor_link_joint" type="fixed">
-      <parent link="sensor_frame_camera_plate_link" />
+    <joint name="sensor_frame_top_beam_link_sensor_frame_sensor_link_joint" type="fixed">
+      <parent link="sensor_frame_top_beam_link" />
       <child link="sensor_frame_sensor_link" />
-      <origin xyz="0.041275 0.041275 0.003175" rpy="0 0 0" />
+      <origin xyz="0.0 0.07 -0.038" rpy="0 ${pi/2.0} ${pi/2.0}" />
     </joint>
     <link name="sensor_frame_sensor_link" />
-    <xacro:kinect2 parent="sensor_frame_sensor_link">
-      <origin xyz="0.009 -0.005 -0.011" rpy="0 0 -0.018" /> <!-- insert calibrated x, y, z, and yaw here -->
-    </xacro:kinect2>
+    <xacro:sensor_asus_xtion_pro parent="sensor_frame_sensor_link">
+      <origin xyz="0.023 -0.014 -0.04" rpy="0.0 -0.223 0.0" /> <!-- insert calibrated x, y, z, pitch, and yaw here -->
+    </xacro:sensor_asus_xtion_pro>
   </xacro:macro>
   <xacro:macro name="nimbus_sensor_frame_calibration" params="parent *origin">
@@ -25,8 +25,8 @@
       <xacro:insert_block name="origin" />
     </xacro:nimbus_sensor_frame_structure>
-    <joint name="sensor_frame_camera_plate_link_sensor_frame_sensor_calibration_link_joint" type="fixed">
-      <parent link="sensor_frame_camera_plate_link" />
+    <joint name="sensor_frame_top_beam_link_sensor_frame_sensor_calibration_link_joint" type="fixed">
+      <parent link="sensor_frame_top_beam_link" />
       <child link="sensor_frame_sensor_calibration_link" />
-      <origin xyz="0.041275 0.041275 0.003175" rpy="0 0 0" />
+      <origin xyz="0.0 0.07 -0.038" rpy="0 ${pi/2.0} ${pi/2.0}" />
     </joint>
     <link name="sensor_frame_sensor_calibration_link" />
@@ -52,6 +52,13 @@
     </joint>
     <link name="sensor_frame_sensor_z_link" />
+    <joint name="sensor_frame_sensor_calibrate_pitch" type="revolute">
+      <parent link="sensor_frame_sensor_z_link" />
+      <child link="sensor_frame_sensor_pitch_link" />
+      <axis xyz="0 1 0" />
+      <limit effort="100" velocity="20" lower="${pi/8}" upper="${-pi/8}" />
+    </joint>
+    <link name="sensor_frame_sensor_pitch_link" />
     <joint name="sensor_frame_sensor_calibrate_yaw" type="revolute">
-      <parent link="sensor_frame_sensor_z_link" />
+      <parent link="sensor_frame_sensor_pitch_link" />
       <child link="sensor_frame_sensor_yaw_link" />
       <axis xyz="0 0 1" />
@@ -64,7 +71,7 @@
     </joint>
     <link name="sensor_frame_sensor_link" />
-    <xacro:kinect2_calibration parent="sensor_frame_sensor_link">
-      <origin xyz="0.009 -0.005 -0.011" rpy="0 0 -0.018" /> <!-- insert calibrated x, y, z, and yaw here -->
-    </xacro:kinect2_calibration>
+    <xacro:sensor_asus_xtion_pro parent="sensor_frame_sensor_link">
+      <origin xyz="0.0 0.0 0.0" rpy="0.0 0.0 0.0" />
+    </xacro:sensor_asus_xtion_pro>
   </xacro:macro>
   <xacro:macro name="nimbus_sensor_frame_structure" params="parent *origin">
@@ -139,42 +146,4 @@
       </collision>
     </link>
-    <joint name="sensor_frame_top_beam_link_sensor_frame_camera_strut_link_joint" type="fixed">
-      <parent link="sensor_frame_top_beam_link" />
-      <child link="sensor_frame_camera_strut_link" />
-      <origin xyz="-0.0254 0.0254 0.0127" rpy="${-pi/4} 0 0" />
-    </joint>
-    <link name="sensor_frame_camera_strut_link">
-      <visual>
-        <geometry>
-          <box size="0.0508 0.1524 0.0254" />
-        </geometry>
-        <origin xyz="0 0.0762 -0.0127" rpy="0 0 0" />
-        <material name="light-gray" />
-      </visual>
-      <collision>
-        <geometry>
-          <box size="0.0808 0.1824 0.0554" />
-        </geometry>
-        <origin xyz="0 0.0762 -0.0127" rpy="0 0 0" />
-      </collision>
-    </link>
-    <joint name="sensor_frame_camera_strut_link_sensor_frame_camera_plate_link_joint" type="fixed">
-      <parent link="sensor_frame_camera_strut_link" />
-      <child link="sensor_frame_camera_plate_link" />
-      <origin xyz="0 0.1016 0.003175" rpy="0 0 0" />
-    </joint>
-    <link name="sensor_frame_camera_plate_link">
-      <visual>
-        <geometry>
-          <box size="0.1016 0.1016 0.00635" />
-        </geometry>
-        <material name="light-gray" />
-      </visual>
-      <collision>
-        <geometry>
-          <box size="0.1316 0.1316 0.01905" />
-        </geometry>
-      </collision>
-    </link>
   </xacro:macro>
   <xacro:macro name="left_bracket" params="parent side">

Commit message: New camera calibration

File: nimbus_description/robots/nimbus.urdf (robot description, URDF)
Before this commit: robot nimbus, 45 links, 44 joints
Joints:
- joint camera_rgb_joint: origin xyz=0.023 -0.014 -0.04 rpy=0.0 -0.223 0.0 -> xyz=0.001 -0.025 0.02 rpy=0.002 -0.236 -0.008

File: nimbus_description/urdf/structure/sensor_structure.urdf.xacro (robot description, xacro)
@@ -18,5 +18,5 @@
     <link name="sensor_frame_sensor_link" />
     <xacro:sensor_asus_xtion_pro parent="sensor_frame_sensor_link">
-      <origin xyz="0.023 -0.014 -0.04" rpy="0.0 -0.223 0.0" /> <!-- insert calibrated x, y, z, pitch, and yaw here -->
+      <origin xyz="0.001 -0.025 0.02" rpy="0.002 -0.236 -0.008" /> <!-- insert calibrated x, y, z, pitch, and yaw here -->
     </xacro:sensor_asus_xtion_pro>
   </xacro:macro>

Commit message: New calibration for a new xtion

File: nimbus_description/robots/nimbus.urdf (robot description, URDF)
Before this commit: robot nimbus, 45 links, 44 joints
Joints:
- joint camera_rgb_joint: origin xyz=0.001 -0.025 0.02 rpy=0.002 -0.236 -0.008 -> xyz=-0.017 0.000 -0.01 rpy=0.003 -0.176 -0.017

File: nimbus_description/urdf/structure/sensor_structure.urdf.xacro (robot description, xacro)
@@ -18,5 +18,7 @@
     <link name="sensor_frame_sensor_link" />
     <xacro:sensor_asus_xtion_pro parent="sensor_frame_sensor_link">
-      <origin xyz="0.001 -0.025 0.02" rpy="0.002 -0.236 -0.008" /> <!-- insert calibrated x, y, z, pitch, and yaw here -->
+      <!--<origin xyz="0.001 -0.025 0.02" rpy="0.002 -0.236 -0.008" />--> <!-- insert calibrated x, y, z, pitch, and yaw here -->
+      <!--<origin xyz="0.007 0.006 0.014" rpy="0.002 -0.228 -0.010" />--> <!-- calbration 200 -->
+      <origin xyz="-0.017 0.000 -0.01" rpy="0.003 -0.176 -0.017" />
     </xacro:sensor_asus_xtion_pro>
   </xacro:macro>

Commit message: renaming point clouds, added satellite camera

File: nimbus_description/robots/nimbus.urdf (robot description, URDF)
Before this commit: robot nimbus, 45 links, 44 joints
Links:
- added link camera_side_link
Joints:
- added joint table_base_link_camera_side_link: type fixed, parent table_base_link, child camera_side_link, origin xyz=-0.104 -0.887 0.252 rpy=-0.032 0.035 1.538
- joint camera_rgb_joint: origin xyz=-0.017 0.000 -0.01 rpy=0.003 -0.176 -0.017 -> xyz=-0.007 0.000 -0.015 rpy=0.003 -0.176 -0.017

File: nimbus_description/robots/nimbus_calibration.urdf (robot description, URDF)
Before this commit: robot nimbus, 51 links, 50 joints
Links:
- added link calibrate_side_camera_link
- added link camera_side_link
- added link camera_side_pitch_link
- added link camera_side_roll_link
- added link camera_side_x_link
- added link camera_side_y_link
- added link camera_side_yaw_link
- added link camera_side_z_link
Joints:
- added joint calibrate_side_camera_link_camera_side_x: type prismatic, parent calibrate_side_camera_link, child camera_side_x_link, axis 1 0 0, limit lower=-0.1 upper=0.1 effort=100 velocity=1
- added joint camera_side_pitch_link_camera_side_yaw_link: type revolute, parent camera_side_pitch_link, child camera_side_yaw_link, axis 0 0 1, limit lower=-0.392699081699 upper=0.392699081699 effort=100 velocity=20
- added joint camera_side_roll_link_camera_side_pitch_link: type revolute, parent camera_side_roll_link, child camera_side_pitch_link, axis 0 1 0, limit lower=-0.392699081699 upper=0.392699081699 effort=100 velocity=20
- added joint camera_side_x_link_camera_side_y_link: type prismatic, parent camera_side_x_link, child camera_side_y_link, axis 0 1 0, limit lower=-0.1 upper=0.1 effort=100 velocity=1
- added joint camera_side_y_link_camera_side_z_link: type prismatic, parent camera_side_y_link, child camera_side_z_link, axis 0 0 1, limit lower=-0.1 upper=0.1 effort=100 velocity=1
- added joint camera_side_yaw_link_camera_side_link: type fixed, parent camera_side_yaw_link, child camera_side_link, origin xyz=0 0 0 rpy=0 0 0
- added joint camera_side_z_link_camera_side_roll_link: type revolute, parent camera_side_z_link, child camera_side_roll_link, axis 1 0 0, limit lower=-0.392699081699 upper=0.392699081699 effort=100 velocity=20
- added joint table_base_link_calibrate_side_camera_link: type fixed, parent table_base_link, child calibrate_side_camera_link, origin xyz=-0.1 -0.9 0.25 rpy=0.0 0.0 1.57079632679

File: nimbus_description/urdf/structure/sensor_structure.urdf.xacro (robot description, xacro)
@@ -8,4 +8,11 @@
   <xacro:property name="pi" value="3.1415926535897931" />
   <xacro:macro name="nimbus_sensor_frame" params="parent *origin">
+    <!-- satellite camera -->
+    <joint name="${parent}_camera_side_link" type="fixed">
+      <parent link="${parent}" />
+      <child link="camera_side_link" />
+      <origin xyz="-0.104 -0.887 0.252" rpy="-0.032 0.035 1.538" /> <!-- Calibrated xyz and rpy for side camera go here (rosrun tf tf_echo /table_base_link /camera_side_link)-->
+    </joint>
+    <link name="camera_side_link" />
     <xacro:nimbus_sensor_frame_structure parent="${parent}">
       <xacro:insert_block name="origin" />
@@ -19,9 +26,65 @@
     <xacro:sensor_asus_xtion_pro parent="sensor_frame_sensor_link">
       <!--<origin xyz="0.001 -0.025 0.02" rpy="0.002 -0.236 -0.008" />--> <!-- insert calibrated x, y, z, pitch, and yaw here -->
-      <!--<origin xyz="0.007 0.006 0.014" rpy="0.002 -0.228 -0.010" />--> <!-- calbration 200 -->
-      <origin xyz="-0.017 0.000 -0.01" rpy="0.003 -0.176 -0.017" />
+      <!--<origin xyz="0.007 0.006 0.014" rpy="0.002 -0.228 -0.010" />--> <!-- calibration 200 -->
+      <!--<origin xyz="-0.017 0.000 -0.01" rpy="0.003 -0.176 -0.017" />-->
+      <origin xyz="-0.007 0.000 -0.015" rpy="0.003 -0.176 -0.017" />
     </xacro:sensor_asus_xtion_pro>
   </xacro:macro>
   <xacro:macro name="nimbus_sensor_frame_calibration" params="parent *origin">
+    <!-- satellite camera -->
+    <joint name="${parent}_calibrate_side_camera_link" type="fixed">
+      <parent link="${parent}" />
+      <child link="calibrate_side_camera_link" />
+      <origin xyz="-0.1 -0.9 0.25" rpy="0.0 0.0 ${pi/2.0}" /> <!-- todo: set to reasonable values -->
+    </joint>
+    <link name="calibrate_side_camera_link" />
+    <joint name="calibrate_side_camera_link_camera_side_x" type="prismatic">
+      <parent link="calibrate_side_camera_link" />
+      <child link="camera_side_x_link" />
+      <axis xyz="1 0 0" />
+      <limit effort="100" velocity="1" lower="-0.1" upper="0.1" />
+    </joint>
+    <link name="camera_side_x_link" />
+    <joint name="camera_side_x_link_camera_side_y_link" type="prismatic">
+      <parent link="camera_side_x_link" />
+      <child link="camera_side_y_link" />
+      <axis xyz="0 1 0" />
+      <limit effort="100" velocity="1" lower="-0.1" upper="0.1" />
+    </joint>
+    <link name="camera_side_y_link" />
+    <joint name="camera_side_y_link_camera_side_z_link" type="prismatic">
+      <parent link="camera_side_y_link" />
+      <child link="camera_side_z_link" />
+      <axis xyz="0 0 1" />
+      <limit effort="100" velocity="1" lower="-0.1" upper="0.1" />
+    </joint>
+    <link name="camera_side_z_link" />
+    <joint name="camera_side_z_link_camera_side_roll_link" type="revolute">
+      <parent link="camera_side_z_link" />
+      <child link="camera_side_roll_link" />
+      <axis xyz="1 0 0" />
+      <limit effort="100" velocity="20" lower="${-pi/8}" upper="${pi/8}" />
+    </joint>
+    <link name="camera_side_roll_link" />
+    <joint name="camera_side_roll_link_camera_side_pitch_link" type="revolute">
+      <parent link="camera_side_roll_link" />
+      <child link="camera_side_pitch_link" />
+      <axis xyz="0 1 0" />
+      <limit effort="100" velocity="20" lower="${-pi/8}" upper="${pi/8}" />
+    </joint>
+    <link name="camera_side_pitch_link" />
+    <joint name="camera_side_pitch_link_camera_side_yaw_link" type="revolute">
+      <parent link="camera_side_pitch_link" />
+      <child link="camera_side_yaw_link" />
+      <axis xyz="0 0 1" />
+      <limit effort="100" velocity="20" lower="${-pi/8}" upper="${pi/8}" />
+    </joint>
+    <link name="camera_side_yaw_link" />
+    <joint name="camera_side_yaw_link_camera_side_link" type="fixed">
+      <parent link="camera_side_yaw_link" />
+      <child link="camera_side_link" />
+      <origin xyz="0 0 0" rpy="0 0 0" />
+    </joint>
+    <link name="camera_side_link"/>
     <xacro:nimbus_sensor_frame_structure parent="${parent}">
       <xacro:insert_block name="origin" />

Commit message: New calibration, testing adjustments to point cloud clicking for the web interface

File: nimbus_description/robots/nimbus.urdf (robot description, URDF)
Before this commit: robot nimbus, 46 links, 45 joints
Joints:
- joint camera_rgb_joint: origin xyz=-0.007 0.000 -0.015 rpy=0.003 -0.176 -0.017 -> xyz=-0.003 -0.025 -0.003 rpy=0.006 -0.224 -0.009
- joint table_base_link_camera_side_link: origin xyz=-0.104 -0.887 0.252 rpy=-0.032 0.035 1.538 -> xyz=-0.152 -1.175 0.328 rpy=-0.019 0.077 1.523

File: nimbus_description/urdf/structure/sensor_structure.urdf.xacro (robot description, xacro)
@@ -12,5 +12,5 @@
       <parent link="${parent}" />
       <child link="camera_side_link" />
-      <origin xyz="-0.104 -0.887 0.252" rpy="-0.032 0.035 1.538" /> <!-- Calibrated xyz and rpy for side camera go here (rosrun tf tf_echo /table_base_link /camera_side_link)-->
+      <origin xyz="-0.152 -1.175 0.328" rpy="-0.019 0.077 1.523" /> <!-- Calibrated xyz and rpy for side camera go here (rosrun tf tf_echo /table_base_link /camera_side_link)-->
     </joint>
     <link name="camera_side_link" />
@@ -25,8 +25,5 @@
     <link name="sensor_frame_sensor_link" />
     <xacro:sensor_asus_xtion_pro parent="sensor_frame_sensor_link">
-      <!--<origin xyz="0.001 -0.025 0.02" rpy="0.002 -0.236 -0.008" />--> <!-- insert calibrated x, y, z, pitch, and yaw here -->
-      <!--<origin xyz="0.007 0.006 0.014" rpy="0.002 -0.228 -0.010" />--> <!-- calibration 200 -->
-      <!--<origin xyz="-0.017 0.000 -0.01" rpy="0.003 -0.176 -0.017" />-->
-      <origin xyz="-0.007 0.000 -0.015" rpy="0.003 -0.176 -0.017" />
+      <origin xyz="-0.003 -0.025 -0.003" rpy="0.006 -0.224 -0.009" /> <!-- insert calibrated x, y, z, pitch, and yaw here (rosrun tf tf_echo /sensor_frame_sensor_calibration_link sensor_frame_sensor_link)-->
     </xacro:sensor_asus_xtion_pro>
   </xacro:macro>
