Commit message: Replaced 6DOF jaco with 7DOF jaco

File: nimbus_description/robots/nimbus.urdf (robot description, URDF)
Before this commit: robot nimbus, 46 links, 45 joints
Links:
- removed link jaco_base_link
- removed link jaco_base_link_simplified
- removed link jaco_ee_link
- removed link jaco_forearm_link
- removed link jaco_forearm_link_simplified
- removed link jaco_shoulder_link
- removed link jaco_upper_arm_link
- removed link jaco_upper_arm_link_simplified
- removed link jaco_wrist_1_link
- removed link jaco_wrist_1_link_simplified
- removed link jaco_wrist_2_link
- removed link jaco_wrist_2_link_simplified
- removed link jaco_wrist_3_link
- removed link jaco_wrist_3_link_simplified
- removed link robotiq_85_base_link
- removed link robotiq_85_left_finger_link
- removed link robotiq_85_left_finger_tip_link
- removed link robotiq_85_left_inner_knuckle_link
- removed link robotiq_85_left_knuckle_link
- removed link robotiq_85_right_finger_link
- removed link robotiq_85_right_finger_tip_link
- removed link robotiq_85_right_inner_knuckle_link
- removed link robotiq_85_right_knuckle_link
- added link j2s7s300_ee_base
- added link j2s7s300_ee_link
- added link j2s7s300_link_1, mass 0.7477; collision mesh filename=package://kinova_description/meshes/shoulder.dae; visual mesh filename=package://kinova_description/meshes/ring_big.STL
- added link j2s7s300_link_2, mass 0.8447; collision mesh filename=package://kinova_description/meshes/arm_half_1.dae; visual mesh filename=package://kinova_description/meshes/arm_half_1.dae
- added link j2s7s300_link_3, mass 0.8447; collision mesh filename=package://kinova_description/meshes/arm_half_2.dae; visual mesh filename=package://kinova_description/meshes/arm_half_2.dae
- added link j2s7s300_link_4, mass 0.6763; collision mesh filename=package://kinova_description/meshes/forearm.dae; visual mesh filename=package://kinova_description/meshes/forearm.dae
- added link j2s7s300_link_5, mass 0.463; collision mesh filename=package://kinova_description/meshes/wrist_spherical_1.dae; visual mesh filename=package://kinova_description/meshes/ring_small.STL
- added link j2s7s300_link_6, mass 0.463; collision mesh filename=package://kinova_description/meshes/wrist_spherical_2.dae; visual mesh filename=package://kinova_description/meshes/ring_small.STL
- added link j2s7s300_link_7; collision mesh filename=package://kinova_description/meshes/wrist_3.stl; visual mesh filename=package://kinova_description/meshes/wrist_3.dae
- added link j2s7s300_link_base, mass 0.46784; collision mesh filename=package://kinova_description/meshes/base.dae; visual mesh filename=package://kinova_description/meshes/base.dae
- added link j2s7s300_robotiq_85_base_link, mass 0.636951; collision mesh filename=package://robotiq_85_description/meshes/collision/robotiq_8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; visual mesh filename=package://robotiq_85_description/meshes/visual/robotiq_85_b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
- added link j2s7s300_robotiq_85_left_finger_link, mass 0.027309; collision mesh filename=package://robotiq_85_description/meshes/collision/robotiq_8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; visual mesh filename=package://robotiq_85_description/meshes/visual/robotiq_85_f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
- added link j2s7s300_robotiq_85_left_finger_tip_link, mass 0.019555; collision mesh filename=package://robotiq_85_description/meshes/collision/robotiq_8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; visual mesh filename=package://robotiq_85_description/meshes/visual/robotiq_85_f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
- added link j2s7s300_robotiq_85_left_inner_knuckle_link, mass 0.029951; collision mesh filename=package://robotiq_85_description/meshes/collision/robotiq_8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; visual mesh filename=package://robotiq_85_description/meshes/visual/robotiq_85_i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
- added link j2s7s300_robotiq_85_left_knuckle_link, mass 0.018491; collision mesh filename=package://robotiq_85_description/meshes/collision/robotiq_8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; visual mesh filename=package://robotiq_85_description/meshes/visual/robotiq_85_k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
- added link j2s7s300_robotiq_85_right_finger_link, mass 0.027309; collision mesh filename=package://robotiq_85_description/meshes/collision/robotiq_8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; visual mesh filename=package://robotiq_85_description/meshes/visual/robotiq_85_f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
- added link j2s7s300_robotiq_85_right_finger_tip_link, mass 0.019555; collision mesh filename=package://robotiq_85_description/meshes/collision/robotiq_8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; visual mesh filename=package://robotiq_85_description/meshes/visual/robotiq_85_f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
- added link j2s7s300_robotiq_85_right_inner_knuckle_link, mass 0.029951; collision mesh filename=package://robotiq_85_description/meshes/collision/robotiq_8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; visual mesh filename=package://robotiq_85_description/meshes/visual/robotiq_85_i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
- added link j2s7s300_robotiq_85_right_knuckle_link, mass 0.018491; collision mesh filename=package://robotiq_85_description/meshes/collision/robotiq_8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; visual mesh filename=package://robotiq_85_description/meshes/visual/robotiq_85_k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
Joints:
- removed joint jaco_base_joint
- removed joint jaco_base_joint_simplified
- removed joint jaco_ee_fixed_joint
- removed joint jaco_elbow_joint
- removed joint jaco_elbow_joint_simplified
- removed joint jaco_shoulder_lift_joint
- removed joint jaco_shoulder_lift_joint_simplified
- removed joint jaco_shoulder_pan_joint
- removed joint jaco_wrist_1_joint
- removed joint jaco_wrist_1_joint_simplified
- removed joint jaco_wrist_2_joint
- removed joint jaco_wrist_2_joint_simplified
- removed joint jaco_wrist_3_joint
- removed joint jaco_wrist_3_joint_simplified
- removed joint robotiq_85_base_joint
- removed joint robotiq_85_left_finger_joint
- removed joint robotiq_85_left_finger_tip_joint
- removed joint robotiq_85_left_inner_knuckle_joint
- removed joint robotiq_85_left_knuckle_joint
- removed joint robotiq_85_right_finger_joint
- removed joint robotiq_85_right_finger_tip_joint
- removed joint robotiq_85_right_inner_knuckle_joint
- removed joint robotiq_85_right_knuckle_joint
- added joint j2s7s300_ee_fixed_joint: type fixed, parent j2s7s300_link_7, child j2s7s300_ee_base, origin xyz=0 0 -0.09380704 rpy=0 1.57079632679 0
- added joint j2s7s300_ee_gripper: type fixed, parent j2s7s300_ee_base, child j2s7s300_ee_link, origin xyz=0.13 0 0
- added joint j2s7s300_joint_1: type continuous, parent j2s7s300_link_base, child j2s7s300_link_1, origin xyz=0 0 0.15675 rpy=0 3.14159265359 0, axis 0 0 1, limit lower=-6.28318530718 upper=6.28318530718 effort=2000 velocity=1
- added joint j2s7s300_joint_2: type revolute, parent j2s7s300_link_1, child j2s7s300_link_2, origin xyz=0 0.0016 -0.11875 rpy=-1.57079632679 0 3.14159265359, axis 0 0 1, limit lower=0.523598775598 upper=5.75958653158 effort=2000 velocity=1
- added joint j2s7s300_joint_3: type continuous, parent j2s7s300_link_2, child j2s7s300_link_3, origin xyz=0 -0.205 0 rpy=-1.57079632679 0 0, axis 0 0 1, limit lower=-6.28318530718 upper=6.28318530718 effort=2000 velocity=1
- added joint j2s7s300_joint_4: type revolute, parent j2s7s300_link_3, child j2s7s300_link_4, origin xyz=0 0 -0.205 rpy=1.57079632679 0 3.14159265359, axis 0 0 1, limit lower=0.523598775598 upper=5.75958653158 effort=2000 velocity=1
- added joint j2s7s300_joint_5: type continuous, parent j2s7s300_link_4, child j2s7s300_link_5, origin xyz=0 0.2073 -0.0114 rpy=-1.57079632679 0 3.14159265359, axis 0 0 1, limit lower=-6.28318530718 upper=6.28318530718 effort=2000 velocity=1
- added joint j2s7s300_joint_6: type revolute, parent j2s7s300_link_5, child j2s7s300_link_6, origin xyz=0 0 -0.10375 rpy=1.57079632679 0 3.14159265359, axis 0 0 1, limit lower=0.523598775598 upper=5.75958653158 effort=2000 velocity=1
- added joint j2s7s300_joint_7: type continuous, parent j2s7s300_link_6, child j2s7s300_link_7, origin xyz=0 0.06075 0 rpy=1.57079632679 0 0, axis 0 0 1, limit effort=600.8 velocity=0.785
- added joint j2s7s300_joint_base: type fixed, parent arm_mount_beam_link, child j2s7s300_link_base, origin xyz=0 0 0 rpy=0 0 0, axis 0 0 0, limit lower=0 upper=0 effort=2000 velocity=1
- added joint j2s7s300_robotiq_85_base_joint: type fixed, parent j2s7s300_ee_base, child j2s7s300_robotiq_85_base_link, origin xyz=0 0 0 rpy=0 0 0
- added joint j2s7s300_robotiq_85_left_finger_joint: type fixed, parent j2s7s300_robotiq_85_left_knuckle_link, child j2s7s300_robotiq_85_left_finger_link, origin xyz=-0.00408552455 -0.03148604435 0.0 rpy=0 0 0
- added joint j2s7s300_robotiq_85_left_finger_tip_joint: type continuous, parent j2s7s300_robotiq_85_left_inner_knuckle_link, child j2s7s300_robotiq_85_left_finger_tip_link, origin xyz=0.04303959807 -0.03759940821 0.0 rpy=0.0 0.0 0.0, axis 0 0 1, limit lower=-3.14 upper=3.14 effort=0.1 velocity=100.0, mimic joint=j2s7s300_robotiq_85_left_knuckle_joint multiplier=-1
- added joint j2s7s300_robotiq_85_left_inner_knuckle_joint: type continuous, parent j2s7s300_robotiq_85_base_link, child j2s7s300_robotiq_85_left_inner_knuckle_link, origin xyz=0.06142 0.0127 0 rpy=3.14159265359 0.0 0.0, axis 0 0 1, limit lower=-3.14 upper=3.14 effort=0.1 velocity=100.0, mimic joint=j2s7s300_robotiq_85_left_knuckle_joint offset=0
- added joint j2s7s300_robotiq_85_left_knuckle_joint: type revolute, parent j2s7s300_robotiq_85_base_link, child j2s7s300_robotiq_85_left_knuckle_link, origin xyz=0.05490451627 0.03060114443 0.0 rpy=3.14159265359 0.0 0.0, axis 0 0 1, limit lower=0.0 upper=0.804 effort=1000 velocity=2.0
- added joint j2s7s300_robotiq_85_right_finger_joint: type fixed, parent j2s7s300_robotiq_85_right_knuckle_link, child j2s7s300_robotiq_85_right_finger_link, origin xyz=-0.00408552455 -0.03148604435 0.0 rpy=0 0 0
- added joint j2s7s300_robotiq_85_right_finger_tip_joint: type continuous, parent j2s7s300_robotiq_85_right_inner_knuckle_link, child j2s7s300_robotiq_85_right_finger_tip_link, origin xyz=0.04303959807 -0.03759940821  0.0 rpy=0.0 0.0 0.0, axis 0 0 1, limit lower=-3.14 upper=3.14 effort=0.1 velocity=100.0, mimic joint=j2s7s300_robotiq_85_left_knuckle_joint multiplier=-1
- added joint j2s7s300_robotiq_85_right_inner_knuckle_joint: type continuous, parent j2s7s300_robotiq_85_base_link, child j2s7s300_robotiq_85_right_inner_knuckle_link, origin xyz=0.06142 -0.0127 0 rpy=0 0 0, axis 0 0 1, limit lower=-3.14 upper=3.14 effort=0.1 velocity=100.0, mimic joint=j2s7s300_robotiq_85_left_knuckle_joint offset=0
- added joint j2s7s300_robotiq_85_right_knuckle_joint: type continuous, parent j2s7s300_robotiq_85_base_link, child j2s7s300_robotiq_85_right_knuckle_link, origin xyz=0.05490451627 -0.03060114443 0.0 rpy=0.0 0.0 0.0, axis 0 0 1, limit lower=-3.14 upper=3.14 effort=1000 velocity=100.0, mimic joint=j2s7s300_robotiq_85_left_knuckle_joint
- joint arm_mount_plate_link_arm_mount_beam_link_joint: origin xyz=0 0 0 rpy=0 0 0 -> xyz=0 0 0 rpy=0 0 3.14159265359
- joint jaco_ee_link_nimbus_ee_link_joint: parent jaco_ee_link -> j2s7s300_ee_link

File: nimbus_description/robots/nimbus_calibration.urdf (robot description, URDF)
Before this commit: robot nimbus, 59 links, 58 joints
Links:
- removed link jaco_base_link
- removed link jaco_base_link_simplified
- removed link jaco_ee_link
- removed link jaco_forearm_link
- removed link jaco_forearm_link_simplified
- removed link jaco_shoulder_link
- removed link jaco_upper_arm_link
- removed link jaco_upper_arm_link_simplified
- removed link jaco_wrist_1_link
- removed link jaco_wrist_1_link_simplified
- removed link jaco_wrist_2_link
- removed link jaco_wrist_2_link_simplified
- removed link jaco_wrist_3_link
- removed link jaco_wrist_3_link_simplified
- removed link robotiq_85_base_link
- removed link robotiq_85_left_finger_link
- removed link robotiq_85_left_finger_tip_link
- removed link robotiq_85_left_inner_knuckle_link
- removed link robotiq_85_left_knuckle_link
- removed link robotiq_85_right_finger_link
- removed link robotiq_85_right_finger_tip_link
- removed link robotiq_85_right_inner_knuckle_link
- removed link robotiq_85_right_knuckle_link
- added link j2s7s300_ee_base
- added link j2s7s300_ee_link
- added link j2s7s300_link_1, mass 0.7477; collision mesh filename=package://kinova_description/meshes/shoulder.dae; visual mesh filename=package://kinova_description/meshes/ring_big.STL
- added link j2s7s300_link_2, mass 0.8447; collision mesh filename=package://kinova_description/meshes/arm_half_1.dae; visual mesh filename=package://kinova_description/meshes/arm_half_1.dae
- added link j2s7s300_link_3, mass 0.8447; collision mesh filename=package://kinova_description/meshes/arm_half_2.dae; visual mesh filename=package://kinova_description/meshes/arm_half_2.dae
- added link j2s7s300_link_4, mass 0.6763; collision mesh filename=package://kinova_description/meshes/forearm.dae; visual mesh filename=package://kinova_description/meshes/forearm.dae
- added link j2s7s300_link_5, mass 0.463; collision mesh filename=package://kinova_description/meshes/wrist_spherical_1.dae; visual mesh filename=package://kinova_description/meshes/ring_small.STL
- added link j2s7s300_link_6, mass 0.463; collision mesh filename=package://kinova_description/meshes/wrist_spherical_2.dae; visual mesh filename=package://kinova_description/meshes/ring_small.STL
- added link j2s7s300_link_7; collision mesh filename=package://kinova_description/meshes/wrist_3.stl; visual mesh filename=package://kinova_description/meshes/wrist_3.dae
- added link j2s7s300_link_base, mass 0.46784; collision mesh filename=package://kinova_description/meshes/base.dae; visual mesh filename=package://kinova_description/meshes/base.dae
- added link j2s7s300_robotiq_85_base_link, mass 0.636951; collision mesh filename=package://robotiq_85_description/meshes/collision/robotiq_8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; visual mesh filename=package://robotiq_85_description/meshes/visual/robotiq_85_b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
- added link j2s7s300_robotiq_85_left_finger_link, mass 0.027309; collision mesh filename=package://robotiq_85_description/meshes/collision/robotiq_8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; visual mesh filename=package://robotiq_85_description/meshes/visual/robotiq_85_f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
- added link j2s7s300_robotiq_85_left_finger_tip_link, mass 0.019555; collision mesh filename=package://robotiq_85_description/meshes/collision/robotiq_8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; visual mesh filename=package://robotiq_85_description/meshes/visual/robotiq_85_f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
- added link j2s7s300_robotiq_85_left_inner_knuckle_link, mass 0.029951; collision mesh filename=package://robotiq_85_description/meshes/collision/robotiq_8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; visual mesh filename=package://robotiq_85_description/meshes/visual/robotiq_85_i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
- added link j2s7s300_robotiq_85_left_knuckle_link, mass 0.018491; collision mesh filename=package://robotiq_85_description/meshes/collision/robotiq_8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; visual mesh filename=package://robotiq_85_description/meshes/visual/robotiq_85_k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
- added link j2s7s300_robotiq_85_right_finger_link, mass 0.027309; collision mesh filename=package://robotiq_85_description/meshes/collision/robotiq_8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; visual mesh filename=package://robotiq_85_description/meshes/visual/robotiq_85_f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
- added link j2s7s300_robotiq_85_right_finger_tip_link, mass 0.019555; collision mesh filename=package://robotiq_85_description/meshes/collision/robotiq_8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; visual mesh filename=package://robotiq_85_description/meshes/visual/robotiq_85_f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
- added link j2s7s300_robotiq_85_right_inner_knuckle_link, mass 0.029951; collision mesh filename=package://robotiq_85_description/meshes/collision/robotiq_8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; visual mesh filename=package://robotiq_85_description/meshes/visual/robotiq_85_i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
- added link j2s7s300_robotiq_85_right_knuckle_link, mass 0.018491; collision mesh filename=package://robotiq_85_description/meshes/collision/robotiq_8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; visual mesh filename=package://robotiq_85_description/meshes/visual/robotiq_85_k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
Joints:
- removed joint jaco_base_joint
- removed joint jaco_base_joint_simplified
- removed joint jaco_ee_fixed_joint
- removed joint jaco_elbow_joint
- removed joint jaco_elbow_joint_simplified
- removed joint jaco_shoulder_lift_joint
- removed joint jaco_shoulder_lift_joint_simplified
- removed joint jaco_shoulder_pan_joint
- removed joint jaco_wrist_1_joint
- removed joint jaco_wrist_1_joint_simplified
- removed joint jaco_wrist_2_joint
- removed joint jaco_wrist_2_joint_simplified
- removed joint jaco_wrist_3_joint
- removed joint jaco_wrist_3_joint_simplified
- removed joint robotiq_85_base_joint
- removed joint robotiq_85_left_finger_joint
- removed joint robotiq_85_left_finger_tip_joint
- removed joint robotiq_85_left_inner_knuckle_joint
- removed joint robotiq_85_left_knuckle_joint
- removed joint robotiq_85_right_finger_joint
- removed joint robotiq_85_right_finger_tip_joint
- removed joint robotiq_85_right_inner_knuckle_joint
- removed joint robotiq_85_right_knuckle_joint
- added joint j2s7s300_ee_fixed_joint: type fixed, parent j2s7s300_link_7, child j2s7s300_ee_base, origin xyz=0 0 -0.09380704 rpy=0 1.57079632679 0
- added joint j2s7s300_ee_gripper: type fixed, parent j2s7s300_ee_base, child j2s7s300_ee_link, origin xyz=0.13 0 0
- added joint j2s7s300_joint_1: type continuous, parent j2s7s300_link_base, child j2s7s300_link_1, origin xyz=0 0 0.15675 rpy=0 3.14159265359 0, axis 0 0 1, limit lower=-6.28318530718 upper=6.28318530718 effort=2000 velocity=1
- added joint j2s7s300_joint_2: type revolute, parent j2s7s300_link_1, child j2s7s300_link_2, origin xyz=0 0.0016 -0.11875 rpy=-1.57079632679 0 3.14159265359, axis 0 0 1, limit lower=0.523598775598 upper=5.75958653158 effort=2000 velocity=1
- added joint j2s7s300_joint_3: type continuous, parent j2s7s300_link_2, child j2s7s300_link_3, origin xyz=0 -0.205 0 rpy=-1.57079632679 0 0, axis 0 0 1, limit lower=-6.28318530718 upper=6.28318530718 effort=2000 velocity=1
- added joint j2s7s300_joint_4: type revolute, parent j2s7s300_link_3, child j2s7s300_link_4, origin xyz=0 0 -0.205 rpy=1.57079632679 0 3.14159265359, axis 0 0 1, limit lower=0.523598775598 upper=5.75958653158 effort=2000 velocity=1
- added joint j2s7s300_joint_5: type continuous, parent j2s7s300_link_4, child j2s7s300_link_5, origin xyz=0 0.2073 -0.0114 rpy=-1.57079632679 0 3.14159265359, axis 0 0 1, limit lower=-6.28318530718 upper=6.28318530718 effort=2000 velocity=1
- added joint j2s7s300_joint_6: type revolute, parent j2s7s300_link_5, child j2s7s300_link_6, origin xyz=0 0 -0.10375 rpy=1.57079632679 0 3.14159265359, axis 0 0 1, limit lower=0.523598775598 upper=5.75958653158 effort=2000 velocity=1
- added joint j2s7s300_joint_7: type continuous, parent j2s7s300_link_6, child j2s7s300_link_7, origin xyz=0 0.06075 0 rpy=1.57079632679 0 0, axis 0 0 1, limit effort=600.8 velocity=0.785
- added joint j2s7s300_joint_base: type fixed, parent arm_mount_beam_link, child j2s7s300_link_base, origin xyz=0 0 0 rpy=0 0 0, axis 0 0 0, limit lower=0 upper=0 effort=2000 velocity=1
- added joint j2s7s300_robotiq_85_base_joint: type fixed, parent j2s7s300_ee_base, child j2s7s300_robotiq_85_base_link, origin xyz=0 0 0 rpy=0 0 0
- added joint j2s7s300_robotiq_85_left_finger_joint: type fixed, parent j2s7s300_robotiq_85_left_knuckle_link, child j2s7s300_robotiq_85_left_finger_link, origin xyz=-0.00408552455 -0.03148604435 0.0 rpy=0 0 0
- added joint j2s7s300_robotiq_85_left_finger_tip_joint: type continuous, parent j2s7s300_robotiq_85_left_inner_knuckle_link, child j2s7s300_robotiq_85_left_finger_tip_link, origin xyz=0.04303959807 -0.03759940821 0.0 rpy=0.0 0.0 0.0, axis 0 0 1, limit lower=-3.14 upper=3.14 effort=0.1 velocity=100.0, mimic joint=j2s7s300_robotiq_85_left_knuckle_joint multiplier=-1
- added joint j2s7s300_robotiq_85_left_inner_knuckle_joint: type continuous, parent j2s7s300_robotiq_85_base_link, child j2s7s300_robotiq_85_left_inner_knuckle_link, origin xyz=0.06142 0.0127 0 rpy=3.14159265359 0.0 0.0, axis 0 0 1, limit lower=-3.14 upper=3.14 effort=0.1 velocity=100.0, mimic joint=j2s7s300_robotiq_85_left_knuckle_joint offset=0
- added joint j2s7s300_robotiq_85_left_knuckle_joint: type revolute, parent j2s7s300_robotiq_85_base_link, child j2s7s300_robotiq_85_left_knuckle_link, origin xyz=0.05490451627 0.03060114443 0.0 rpy=3.14159265359 0.0 0.0, axis 0 0 1, limit lower=0.0 upper=0.804 effort=1000 velocity=2.0
- added joint j2s7s300_robotiq_85_right_finger_joint: type fixed, parent j2s7s300_robotiq_85_right_knuckle_link, child j2s7s300_robotiq_85_right_finger_link, origin xyz=-0.00408552455 -0.03148604435 0.0 rpy=0 0 0
- added joint j2s7s300_robotiq_85_right_finger_tip_joint: type continuous, parent j2s7s300_robotiq_85_right_inner_knuckle_link, child j2s7s300_robotiq_85_right_finger_tip_link, origin xyz=0.04303959807 -0.03759940821  0.0 rpy=0.0 0.0 0.0, axis 0 0 1, limit lower=-3.14 upper=3.14 effort=0.1 velocity=100.0, mimic joint=j2s7s300_robotiq_85_left_knuckle_joint multiplier=-1
- added joint j2s7s300_robotiq_85_right_inner_knuckle_joint: type continuous, parent j2s7s300_robotiq_85_base_link, child j2s7s300_robotiq_85_right_inner_knuckle_link, origin xyz=0.06142 -0.0127 0 rpy=0 0 0, axis 0 0 1, limit lower=-3.14 upper=3.14 effort=0.1 velocity=100.0, mimic joint=j2s7s300_robotiq_85_left_knuckle_joint offset=0
- added joint j2s7s300_robotiq_85_right_knuckle_joint: type continuous, parent j2s7s300_robotiq_85_base_link, child j2s7s300_robotiq_85_right_knuckle_link, origin xyz=0.05490451627 -0.03060114443 0.0 rpy=0.0 0.0 0.0, axis 0 0 1, limit lower=-3.14 upper=3.14 effort=1000 velocity=100.0, mimic joint=j2s7s300_robotiq_85_left_knuckle_joint
- joint arm_mount_plate_link_arm_mount_beam_link_joint: origin xyz=0 0 0 rpy=0 0 0 -> xyz=0 0 0 rpy=0 0 3.14159265359
- joint jaco_ee_link_nimbus_ee_link_joint: parent jaco_ee_link -> j2s7s300_ee_link

File: nimbus_description/urdf/structure/arm_mount.urdf.xacro (robot description, xacro)
@@ -1,6 +1,6 @@
 <?xml version="1.0"?>
 <robot xmlns:xacro="http://www.ros.org/wiki/xacro">
-  <xacro:include filename="$(find jaco2_description)/urdf/jaco.urdf.xacro" />
-  <xacro:include filename="$(find nimbus_description)/urdf/structure/arm_simplified.xacro" />
+  <xacro:include filename="$(find nimbus_description)/urdf/structure/arm_simplified.xacro" />-->
+  <xacro:include filename="$(find kinova_description)/urdf/j2s7s300.xacro" />
   <!-- Xacro properties -->
   <xacro:property name="M_PI" value="3.1415926535897931" />
@@ -31,5 +31,5 @@
       <parent link="arm_mount_plate_link" />
       <child link="arm_mount_beam_link" />
-      <origin xyz="0 0 0" rpy="0 0 0" />
+      <origin xyz="0 0 0" rpy="0 0 ${pi}" />
     </joint>
     <link name="arm_mount_beam_link">
@@ -48,10 +48,7 @@
       </collision>
     </link>
-    <xacro:jaco2_arm prefix="jaco_" parent="arm_mount_beam_link">
-      <origin xyz="0 0 0.0508" rpy="0 0 ${pi}" />
-    </xacro:jaco2_arm>
-    <xacro:jaco_arm_simplified prefix="jaco_" />
+    <xacro:j2s7s300 base_parent="arm_mount_beam_link"></xacro:j2s7s300>
     <joint name="jaco_ee_link_nimbus_ee_link_joint" type="fixed">
-      <parent link="jaco_ee_link" />
+      <parent link="j2s7s300_ee_link" />
       <child link="nimbus_ee_link" />
       <origin xyz="0 0 0" rpy="0 ${-pi/2.0} 0" />
