Commit message: Lots of small adjustments to get the nimbus crowd interface working smoothly

File: nimbus_description/robots/nimbus.urdf (robot description, URDF)
Before this commit: robot nimbus, 42 links, 41 joints
Links:
- removed link j2s7s300_robotiq_85_base_link
- removed link j2s7s300_robotiq_85_left_finger_link
- removed link j2s7s300_robotiq_85_left_finger_tip_link
- removed link j2s7s300_robotiq_85_left_inner_knuckle_link
- removed link j2s7s300_robotiq_85_left_knuckle_link
- removed link j2s7s300_robotiq_85_right_finger_link
- removed link j2s7s300_robotiq_85_right_finger_tip_link
- removed link j2s7s300_robotiq_85_right_inner_knuckle_link
- removed link j2s7s300_robotiq_85_right_knuckle_link
- added link arm_mount_offset_link
- added link robotiq_85_base_link, mass 0.636951; collision mesh filename=package://robotiq_85_description/meshes/collision/robotiq_8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; visual mesh filename=package://robotiq_85_description/meshes/visual/robotiq_85_b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
- added link robotiq_85_left_finger_link, mass 0.027309; collision mesh filename=package://robotiq_85_description/meshes/collision/robotiq_8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; visual mesh filename=package://robotiq_85_description/meshes/visual/robotiq_85_f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
- added link robotiq_85_left_finger_tip_link, mass 0.019555; collision mesh filename=package://robotiq_85_description/meshes/collision/robotiq_8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; visual mesh filename=package://robotiq_85_description/meshes/visual/robotiq_85_f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
- added link robotiq_85_left_inner_knuckle_link, mass 0.029951; collision mesh filename=package://robotiq_85_description/meshes/collision/robotiq_8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; visual mesh filename=package://robotiq_85_description/meshes/visual/robotiq_85_i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
- added link robotiq_85_left_knuckle_link, mass 0.018491; collision mesh filename=package://robotiq_85_description/meshes/collision/robotiq_8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; visual mesh filename=package://robotiq_85_description/meshes/visual/robotiq_85_k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
- added link robotiq_85_right_finger_link, mass 0.027309; collision mesh filename=package://robotiq_85_description/meshes/collision/robotiq_8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; visual mesh filename=package://robotiq_85_description/meshes/visual/robotiq_85_f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
- added link robotiq_85_right_finger_tip_link, mass 0.019555; collision mesh filename=package://robotiq_85_description/meshes/collision/robotiq_8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; visual mesh filename=package://robotiq_85_description/meshes/visual/robotiq_85_f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
- added link robotiq_85_right_inner_knuckle_link, mass 0.029951; collision mesh filename=package://robotiq_85_description/meshes/collision/robotiq_8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; visual mesh filename=package://robotiq_85_description/meshes/visual/robotiq_85_i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
- added link robotiq_85_right_knuckle_link, mass 0.018491; collision mesh filename=package://robotiq_85_description/meshes/collision/robotiq_8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; visual mesh filename=package://robotiq_85_description/meshes/visual/robotiq_85_k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
- added link sensor_frame_left_support_link; collision box size=0.0454 0.4572 0.4572; visual box size=0.0254 0.4572 0.4572
- added link sensor_frame_right_support_link; collision box size=0.0454 0.4572 0.4572; visual box size=0.0254 0.4572 0.4572
Joints:
- removed joint j2s7s300_robotiq_85_base_joint
- removed joint j2s7s300_robotiq_85_left_finger_joint
- removed joint j2s7s300_robotiq_85_left_finger_tip_joint
- removed joint j2s7s300_robotiq_85_left_inner_knuckle_joint
- removed joint j2s7s300_robotiq_85_left_knuckle_joint
- removed joint j2s7s300_robotiq_85_right_finger_joint
- removed joint j2s7s300_robotiq_85_right_finger_tip_joint
- removed joint j2s7s300_robotiq_85_right_inner_knuckle_joint
- removed joint j2s7s300_robotiq_85_right_knuckle_joint
- added joint arm_mount_beam_link_arm_mount_offset_link_joint: type fixed, parent arm_mount_beam_link, child arm_mount_offset_link, origin xyz=0 0 0.0508 rpy=0 0 3.14159265359
- added joint robotiq_85_base_joint: type fixed, parent j2s7s300_ee_base, child robotiq_85_base_link, origin xyz=0 0 0 rpy=0 0 0
- added joint robotiq_85_left_finger_joint: type fixed, parent robotiq_85_left_knuckle_link, child robotiq_85_left_finger_link, origin xyz=-0.00408552455 -0.03148604435 0.0 rpy=0 0 0
- added joint robotiq_85_left_finger_tip_joint: type continuous, parent robotiq_85_left_inner_knuckle_link, child robotiq_85_left_finger_tip_link, origin xyz=0.04303959807 -0.03759940821 0.0 rpy=0.0 0.0 0.0, axis 0 0 1, limit lower=-3.14 upper=3.14 effort=0.1 velocity=100.0, mimic joint=robotiq_85_left_knuckle_joint multiplier=-1
- added joint robotiq_85_left_inner_knuckle_joint: type continuous, parent robotiq_85_base_link, child robotiq_85_left_inner_knuckle_link, origin xyz=0.06142 0.0127 0 rpy=3.14159265359 0.0 0.0, axis 0 0 1, limit lower=-3.14 upper=3.14 effort=0.1 velocity=100.0, mimic joint=robotiq_85_left_knuckle_joint offset=0
- added joint robotiq_85_left_knuckle_joint: type revolute, parent robotiq_85_base_link, child robotiq_85_left_knuckle_link, origin xyz=0.05490451627 0.03060114443 0.0 rpy=3.14159265359 0.0 0.0, axis 0 0 1, limit lower=0.0 upper=0.804 effort=1000 velocity=2.0
- added joint robotiq_85_right_finger_joint: type fixed, parent robotiq_85_right_knuckle_link, child robotiq_85_right_finger_link, origin xyz=-0.00408552455 -0.03148604435 0.0 rpy=0 0 0
- added joint robotiq_85_right_finger_tip_joint: type continuous, parent robotiq_85_right_inner_knuckle_link, child robotiq_85_right_finger_tip_link, origin xyz=0.04303959807 -0.03759940821  0.0 rpy=0.0 0.0 0.0, axis 0 0 1, limit lower=-3.14 upper=3.14 effort=0.1 velocity=100.0, mimic joint=robotiq_85_left_knuckle_joint multiplier=-1
- added joint robotiq_85_right_inner_knuckle_joint: type continuous, parent robotiq_85_base_link, child robotiq_85_right_inner_knuckle_link, origin xyz=0.06142 -0.0127 0 rpy=0 0 0, axis 0 0 1, limit lower=-3.14 upper=3.14 effort=0.1 velocity=100.0, mimic joint=robotiq_85_left_knuckle_joint offset=0
- added joint robotiq_85_right_knuckle_joint: type continuous, parent robotiq_85_base_link, child robotiq_85_right_knuckle_link, origin xyz=0.05490451627 -0.03060114443 0.0 rpy=0.0 0.0 0.0, axis 0 0 1, limit lower=-3.14 upper=3.14 effort=1000 velocity=100.0, mimic joint=robotiq_85_left_knuckle_joint
- added joint sensor_frame_left_strut_link_sensor_frame_left_support_link_joint: type fixed, parent sensor_frame_left_strut_link, child sensor_frame_left_support_link, origin xyz=0 0.2286 0.2286 rpy=0 0 0
- added joint sensor_frame_right_strut_link_sensor_frame_right_support_link_joint: type fixed, parent sensor_frame_right_strut_link, child sensor_frame_right_support_link, origin xyz=0 0.2286 0.2286 rpy=0 0 0
- joint arm_mount_plate_link_arm_mount_beam_link_joint: origin xyz=0 0 0 rpy=0 0 3.14159265359 -> xyz=0 0 0 rpy=0 0 0
- joint j2s7s300_joint_base: parent arm_mount_beam_link -> arm_mount_offset_link
- joint jaco_ee_link_nimbus_ee_link_joint: origin xyz=0 0 0 rpy=0 -1.57079632679 0 -> xyz=0 0 0 rpy=1.57079632679 0 0

File: nimbus_description/robots/nimbus_calibration.urdf (robot description, URDF)
Before this commit: robot nimbus, 55 links, 54 joints
Links:
- removed link j2s7s300_robotiq_85_base_link
- removed link j2s7s300_robotiq_85_left_finger_link
- removed link j2s7s300_robotiq_85_left_finger_tip_link
- removed link j2s7s300_robotiq_85_left_inner_knuckle_link
- removed link j2s7s300_robotiq_85_left_knuckle_link
- removed link j2s7s300_robotiq_85_right_finger_link
- removed link j2s7s300_robotiq_85_right_finger_tip_link
- removed link j2s7s300_robotiq_85_right_inner_knuckle_link
- removed link j2s7s300_robotiq_85_right_knuckle_link
- added link arm_mount_offset_link
- added link robotiq_85_base_link, mass 0.636951; collision mesh filename=package://robotiq_85_description/meshes/collision/robotiq_8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; visual mesh filename=package://robotiq_85_description/meshes/visual/robotiq_85_b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
- added link robotiq_85_left_finger_link, mass 0.027309; collision mesh filename=package://robotiq_85_description/meshes/collision/robotiq_8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; visual mesh filename=package://robotiq_85_description/meshes/visual/robotiq_85_f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
- added link robotiq_85_left_finger_tip_link, mass 0.019555; collision mesh filename=package://robotiq_85_description/meshes/collision/robotiq_8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; visual mesh filename=package://robotiq_85_description/meshes/visual/robotiq_85_f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
- added link robotiq_85_left_inner_knuckle_link, mass 0.029951; collision mesh filename=package://robotiq_85_description/meshes/collision/robotiq_8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; visual mesh filename=package://robotiq_85_description/meshes/visual/robotiq_85_i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
- added link robotiq_85_left_knuckle_link, mass 0.018491; collision mesh filename=package://robotiq_85_description/meshes/collision/robotiq_8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; visual mesh filename=package://robotiq_85_description/meshes/visual/robotiq_85_k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
- added link robotiq_85_right_finger_link, mass 0.027309; collision mesh filename=package://robotiq_85_description/meshes/collision/robotiq_8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; visual mesh filename=package://robotiq_85_description/meshes/visual/robotiq_85_f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
- added link robotiq_85_right_finger_tip_link, mass 0.019555; collision mesh filename=package://robotiq_85_description/meshes/collision/robotiq_8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; visual mesh filename=package://robotiq_85_description/meshes/visual/robotiq_85_f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
- added link robotiq_85_right_inner_knuckle_link, mass 0.029951; collision mesh filename=package://robotiq_85_description/meshes/collision/robotiq_8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; visual mesh filename=package://robotiq_85_description/meshes/visual/robotiq_85_i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
- added link robotiq_85_right_knuckle_link, mass 0.018491; collision mesh filename=package://robotiq_85_description/meshes/collision/robotiq_8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; visual mesh filename=package://robotiq_85_description/meshes/visual/robotiq_85_k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
- added link sensor_frame_left_support_link; collision box size=0.0454 0.4572 0.4572; visual box size=0.0254 0.4572 0.4572
- added link sensor_frame_right_support_link; collision box size=0.0454 0.4572 0.4572; visual box size=0.0254 0.4572 0.4572
Joints:
- removed joint j2s7s300_robotiq_85_base_joint
- removed joint j2s7s300_robotiq_85_left_finger_joint
- removed joint j2s7s300_robotiq_85_left_finger_tip_joint
- removed joint j2s7s300_robotiq_85_left_inner_knuckle_joint
- removed joint j2s7s300_robotiq_85_left_knuckle_joint
- removed joint j2s7s300_robotiq_85_right_finger_joint
- removed joint j2s7s300_robotiq_85_right_finger_tip_joint
- removed joint j2s7s300_robotiq_85_right_inner_knuckle_joint
- removed joint j2s7s300_robotiq_85_right_knuckle_joint
- added joint arm_mount_beam_link_arm_mount_offset_link_joint: type fixed, parent arm_mount_beam_link, child arm_mount_offset_link, origin xyz=0 0 0.0508 rpy=0 0 3.14159265359
- added joint robotiq_85_base_joint: type fixed, parent j2s7s300_ee_base, child robotiq_85_base_link, origin xyz=0 0 0 rpy=0 0 0
- added joint robotiq_85_left_finger_joint: type fixed, parent robotiq_85_left_knuckle_link, child robotiq_85_left_finger_link, origin xyz=-0.00408552455 -0.03148604435 0.0 rpy=0 0 0
- added joint robotiq_85_left_finger_tip_joint: type continuous, parent robotiq_85_left_inner_knuckle_link, child robotiq_85_left_finger_tip_link, origin xyz=0.04303959807 -0.03759940821 0.0 rpy=0.0 0.0 0.0, axis 0 0 1, limit lower=-3.14 upper=3.14 effort=0.1 velocity=100.0, mimic joint=robotiq_85_left_knuckle_joint multiplier=-1
- added joint robotiq_85_left_inner_knuckle_joint: type continuous, parent robotiq_85_base_link, child robotiq_85_left_inner_knuckle_link, origin xyz=0.06142 0.0127 0 rpy=3.14159265359 0.0 0.0, axis 0 0 1, limit lower=-3.14 upper=3.14 effort=0.1 velocity=100.0, mimic joint=robotiq_85_left_knuckle_joint offset=0
- added joint robotiq_85_left_knuckle_joint: type revolute, parent robotiq_85_base_link, child robotiq_85_left_knuckle_link, origin xyz=0.05490451627 0.03060114443 0.0 rpy=3.14159265359 0.0 0.0, axis 0 0 1, limit lower=0.0 upper=0.804 effort=1000 velocity=2.0
- added joint robotiq_85_right_finger_joint: type fixed, parent robotiq_85_right_knuckle_link, child robotiq_85_right_finger_link, origin xyz=-0.00408552455 -0.03148604435 0.0 rpy=0 0 0
- added joint robotiq_85_right_finger_tip_joint: type continuous, parent robotiq_85_right_inner_knuckle_link, child robotiq_85_right_finger_tip_link, origin xyz=0.04303959807 -0.03759940821  0.0 rpy=0.0 0.0 0.0, axis 0 0 1, limit lower=-3.14 upper=3.14 effort=0.1 velocity=100.0, mimic joint=robotiq_85_left_knuckle_joint multiplier=-1
- added joint robotiq_85_right_inner_knuckle_joint: type continuous, parent robotiq_85_base_link, child robotiq_85_right_inner_knuckle_link, origin xyz=0.06142 -0.0127 0 rpy=0 0 0, axis 0 0 1, limit lower=-3.14 upper=3.14 effort=0.1 velocity=100.0, mimic joint=robotiq_85_left_knuckle_joint offset=0
- added joint robotiq_85_right_knuckle_joint: type continuous, parent robotiq_85_base_link, child robotiq_85_right_knuckle_link, origin xyz=0.05490451627 -0.03060114443 0.0 rpy=0.0 0.0 0.0, axis 0 0 1, limit lower=-3.14 upper=3.14 effort=1000 velocity=100.0, mimic joint=robotiq_85_left_knuckle_joint
- added joint sensor_frame_left_strut_link_sensor_frame_left_support_link_joint: type fixed, parent sensor_frame_left_strut_link, child sensor_frame_left_support_link, origin xyz=0 0.2286 0.2286 rpy=0 0 0
- added joint sensor_frame_right_strut_link_sensor_frame_right_support_link_joint: type fixed, parent sensor_frame_right_strut_link, child sensor_frame_right_support_link, origin xyz=0 0.2286 0.2286 rpy=0 0 0
- joint arm_mount_plate_link_arm_mount_beam_link_joint: origin xyz=0 0 0 rpy=0 0 3.14159265359 -> xyz=0 0 0 rpy=0 0 0
- joint j2s7s300_joint_base: parent arm_mount_beam_link -> arm_mount_offset_link
- joint jaco_ee_link_nimbus_ee_link_joint: origin xyz=0 0 0 rpy=0 -1.57079632679 0 -> xyz=0 0 0 rpy=1.57079632679 0 0

File: nimbus_description/urdf/structure/sensor_structure.urdf.xacro (robot description, xacro)
@@ -168,4 +168,26 @@
     <xacro:left_bracket parent="sensor_frame_left_strut_link" side="left" />
     <xacro:right_bracket parent="sensor_frame_left_strut_link" side="left" />
+    <joint name="sensor_frame_left_strut_link_sensor_frame_left_support_link_joint" type="fixed">
+      <parent link="sensor_frame_left_strut_link" />
+      <child link="sensor_frame_left_support_link" />
+      <origin xyz="0 0.2286 0.2286" rpy="0 0 0" />
+    </joint>
+    <link name="sensor_frame_left_support_link" >
+      <visual>
+        <geometry>
+          <box size="0.0254 0.4572 0.4572" />
+        </geometry>
+        <origin xyz="0 0 0" rpy="0 0 0" />
+        <material name="light-gray">
+          <color rgba="0.4 0.4 0.4 1" />
+        </material>
+      </visual>
+      <collision>
+        <geometry>
+          <box size="0.0454 0.4572 0.4572" />
+        </geometry>
+        <origin xyz="0 0 0" rpy="0 0 0" />
+      </collision>
+    </link>
     <joint name="sensor_frame_center_link_sensor_frame_right_strut_link_joint" type="fixed">
       <parent link="sensor_frame_center_link" />
@@ -190,4 +212,26 @@
     <xacro:left_bracket parent="sensor_frame_right_strut_link" side="right" />
     <xacro:right_bracket parent="sensor_frame_right_strut_link" side="right" />
+    <joint name="sensor_frame_right_strut_link_sensor_frame_right_support_link_joint" type="fixed">
+      <parent link="sensor_frame_right_strut_link" />
+      <child link="sensor_frame_right_support_link" />
+      <origin xyz="0 0.2286 0.2286" rpy="0 0 0" />
+    </joint>
+    <link name="sensor_frame_right_support_link" >
+      <visual>
+        <geometry>
+          <box size="0.0254 0.4572 0.4572" />
+        </geometry>
+        <origin xyz="0 0 0" rpy="0 0 0" />
+        <material name="light-gray">
+          <color rgba="0.4 0.4 0.4 1" />
+        </material>
+      </visual>
+      <collision>
+        <geometry>
+          <box size="0.0454 0.4572 0.4572" />
+        </geometry>
+        <origin xyz="0 0 0" rpy="0 0 0" />
+      </collision>
+    </link>
     <joint name="sensor_frame_center_link_sensor_frame_top_beam_link_joint" type="fixed">
       <parent link="sensor_frame_center_link" />
